Commit message: fix 4

File: ar_tags/models/1234tag.urdf (robot description, URDF)
Before this commit: robot my_ar_tag, 2 links, 1 joints
Links:
- removed link link
- added link base_link; visual box size=1 1 1
Joints:
- removed joint world_to_link
- added joint world_to_base_link: type fixed, parent world, child base_link, origin xyz=0 0 0.5 rpy=0 0 0

Commit message: fix 5

File: ar_tags/models/1234tag.urdf (robot description, URDF)
Before this commit: robot simple_box, 2 links, 1 joints
Links:
- removed link base_link
- added link link; visual mesh filename=package://ar_tags/models/1234tag.dae scale=1 1 1

Commit message: fix 6

File: ar_tags/models/1234tag.urdf (robot description, URDF)
Before this commit: robot my_ar_tag, 2 links, 1 joints
Links:
- link link: geometry visual mesh filename=package://fetch_test/ar_tags/models/1234tag.dae scale=1 1 1

Commit message: fix 8

File: ar_tags/models/1234tag.urdf (robot description, URDF)
Before this commit: robot my_ar_tag, 2 links, 1 joints
Links:
- link link: geometry visual mesh filename=file:///home/catkin_ws/src/fetch-test/ar_tags/models/1234ta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 scale=1 1 1

Commit message: fix 9

File: ar_tags/models/1234tag.urdf (robot description, URDF)
Before this commit: robot my_ar_tag, 2 links, 1 joints
Links:
- removed link link
- added link base_link; visual mesh filename=file:///home/catkin_ws/src/fetch-test/ar_tags/models/1234ta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 scale=1 1 1

Commit message: collisions and static

File: ar_tags/models/1234tag.urdf (robot description, URDF)
Before this commit: robot my_ar_tag, 2 links, 1 joints
Links:
- link base_link: geometry collision mesh filename=file:///home/catkin_ws/src/fetch-test/ar_tags/models/1234ta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 scale=1 1 1; visual mesh filename=file:///home/catkin_ws/src/fetch-test/ar_tags/models/1234ta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 scale=1 1 1
